File: 011/011.kicad_pcb (KiCad board)
At the start: 2 copper layers, 25.3 x 22 mm, 8 parts, among them J2 Conn_01x14

Commit message: Final, EOL Commit
Parts:
- removed 001 LED: Bridge for 001, Resistor_SMD:R_0201_0603Metric
- removed G***: LOGO, MSL0104RGB:3.5mm CC_Logo
- removed J2: Conn_01x14, Molex 503480-1400:503480-1400
Routing:
- net /Annode: track 33.0 -> 24.3 mm
- net VCC: track 27.1 -> 18.8 mm, vias 2 -> 1
- net /R: track 19.3 -> 17.5 mm, vias 2 -> 0
- net GND: track 1.29 -> 0.00 mm, vias 44 -> 48
- net /d+: track 21.2 -> 20.7 mm
Other:
- net class Default removed
- board text added: "JDS-011 V1.2"
- board text removed: "JDS-001/011 V1.1"

Commit message: Updated 011 gerbers
Connections:
- USB pad S1: GND -> (no net)
Routing:
- net /d-: track 19.9 -> 20.7 mm
- net /d+: track 20.7 -> 21.5 mm
- net GND: vias 48 -> 51
Changed lines of the file:
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@@
     (pad "B12" smd rect locked (at -3.25 4.045) (size 0.6 1.45) (layers "B.Cu" "B.Paste" "B.Mask")
       (net 1 "GND"))
-    (pad "S1" thru_hole oval locked (at -4.32 3.13) (size 1 2.1) (drill oval 0.6 1.7) (layers *.Cu *.Mask)
-      (net 1 "GND"))
-    (pad "S1" thru_hole oval locked (at 4.32 -1.05) (size 1 1.6) (drill oval 0.6 1.2) (layers *.Cu *.Mask)
-      (net 1 "GND"))
-    (pad "S1" thru_hole oval locked (at -4.32 -1.05) (size 1 1.6) (drill oval 0.6 1.2) (layers *.Cu *.Mask)
-      (net 1 "GND"))
-    (pad "S1" thru_hole oval locked (at 4.32 3.13) (size 1 2.1) (drill oval 0.6 1.7) (layers *.Cu *.Mask)
-      (net 1 "GND"))
+    (pad "S1" thru_hole oval locked (at -4.32 3.13) (size 1 2.1) (drill oval 0.6 1.7) (layers *.Cu *.Mask))
+    (pad "S1" thru_hole oval locked (at 4.32 -1.05) (size 1 1.6) (drill oval 0.6 1.2) (layers *.Cu *.Mask))
+    (pad "S1" thru_hole oval locked (at -4.32 -1.05) (size 1 1.6) (drill oval 0.6 1.2) (layers *.Cu *.Mask))
+    (pad "S1" thru_hole oval locked (at 4.32 3.13) (size 1 2.1) (drill oval 0.6 1.7) (layers *.Cu *.Mask))
     (model "${KISYS3DMOD}/Connector_USB.3dshapes/USB_C_Receptacle_HRO_TYPE-C-31-M-12.wrl"
       (offset (xyz 0 0 0))
@@
     )
   )
+  (gr_poly
+    (pts
+      (xy 108.0262 58.802399)
+      (xy 107.2642 58.802399)
+      (xy 107.2642 57.946798)
+      (xy 108.0262 57.946798)
+    ) (layer "F.Cu") (width 0.0001) (fill solid))
   (gr_line (start 129.413 64.389) (end 129.413 53.34) (layer "Edge.Cuts") (width 0.05))
   (gr_line (start 104.14 64.3255) (end 110.4265 64.3255) (layer "Edge.Cuts") (width 0.05))
@@
   (via (at 113.538 63.881) (size 0.4) (drill 0.3) (layers "F.Cu" "B.Cu") (net 1))
   (via (at 107.42 63.56) (size 0.4) (drill 0.3) (layers "F.Cu" "B.Cu") (net 1))
+  (via (at 117.856 70.9168) (size 0.4) (drill 0.3) (layers "F.Cu" "B.Cu") (free) (net 1))
   (via (at 120.015 61.087) (size 0.4) (drill 0.3) (layers "F.Cu" "B.Cu") (net 1))
   (via (at 112.268 59.944) (size 0.4) (drill 0.3) (layers "F.Cu" "B.Cu") (net 1))
   (via (at 114.046 56.388) (size 0.4) (drill 0.3) (layers "F.Cu" "B.Cu") (net 1))
   (via (at 122.047 66.675) (size 0.4) (drill 0.3) (layers "F.Cu" "B.Cu") (net 1))
-  (via (at 114.427 58.674) (size 0.4) (drill 0.3) (layers "F.Cu" "B.Cu") (net 1))
   (via (at 114.554 55.753) (size 0.4) (drill 0.3) (layers "F.Cu" "B.Cu") (net 1))
   (via (at 118.8212 73.4568) (size 0.4) (drill 0.3) (layers "F.Cu" "B.Cu") (free) (net 1))
   (via (at 120.904 62.738) (size 0.4) (drill 0.3) (layers "F.Cu" "B.Cu") (net 1))
-  (via (at 113.665 59.436) (size 0.4) (drill 0.3) (layers "F.Cu" "B.Cu") (net 1))
   (via (at 116.459 57.277) (size 0.4) (drill 0.3) (layers "F.Cu" "B.Cu") (net 1))
   (via (at 117.094 67.437) (size 0.4) (drill 0.3) (layers "F.Cu" "B.Cu") (net 1))
@@
   (via (at 121.158 58.039) (size 0.4) (drill 0.3) (layers "F.Cu" "B.Cu") (net 1))
   (via (at 115.443 65.786) (size 0.4) (drill 0.3) (layers "F.Cu" "B.Cu") (net 1))
+  (via (at 120.2436 73.9648) (size 0.4) (drill 0.3) (layers "F.Cu" "B.Cu") (free) (net 1))
   (via (at 105.11 63.46) (size 0.4) (drill 0.3) (layers "F.Cu" "B.Cu") (net 1))
   (via (at 119.888 55.499) (size 0.4) (drill 0.3) (layers "F.Cu" "B.Cu") (net 1))
   (via (at 106.8324 60.6298) (size 0.4) (drill 0.3) (layers "F.Cu" "B.Cu") (free) (net 1))
   (via (at 122.428 56.769) (size 0.4) (drill 0.3) (layers "F.Cu" "B.Cu") (net 1))
+  (via (at 118.1608 69.4436) (size 0.4) (drill 0.3) (layers "F.Cu" "B.Cu") (free) (net 1))
   (via (at 115.062 61.595) (size 0.4) (drill 0.3) (layers "F.Cu" "B.Cu") (net 1))
   (via (at 106.807 59.055) (size 0.4) (drill 0.3) (layers "F.Cu" "B.Cu") (net 1))
@@
   (via (at 110.8202 57.0738) (size 0.4) (drill 0.3) (layers "F.Cu" "B.Cu") (net 1))
   (via (at 119.253 62.23) (size 0.4) (drill 0.3) (layers "F.Cu" "B.Cu") (net 1))
+  (via (at 116.713 74.2442) (size 0.4) (drill 0.3) (layers "F.Cu" "B.Cu") (free) (net 1))
+  (via (at 116.205 70.6374) (size 0.4) (drill 0.3) (layers "F.Cu" "B.Cu") (free) (net 1))
   (via (at 123.825 62.865) (size 0.4) (drill 0.3) (layers "F.Cu" "B.Cu") (net 1))
   (via (at 116.967 61.976) (size 0.4) (drill 0.3) (layers "F.Cu" "B.Cu") (net 1))
@@
   (segment (start 118.6549 55.5891) (end 118.999 55.245) (width 0.2) (layer "B.Cu") (net 4))
   (segment (start 118.6549 59.5159) (end 118.6549 55.5891) (width 0.2) (layer "B.Cu") (net 4))
+  (segment (start 108.216701 57.1246) (end 107.6452 57.1246) (width 0.2) (layer "F.Cu") (net 6))
+  (segment (start 119.413801 56.613) (end 115.4092 56.613) (width 0.2) (layer "F.Cu") (net 6))
+  (segment (start 119.65819 56.99881) (end 119.65819 56.857389) (width 0.2) (layer "F.Cu") (net 6))
   (segment (start 111.201002 59.153) (end 109.147601 57.099599) (width 0.2) (layer "F.Cu") (net 6))
-  (segment (start 115.4092 56.613) (end 112.8692 59.153) (width 0.2) (layer "F.Cu") (net 6))
-  (segment (start 119.65819 56.99881) (end 119.65819 56.857389) (width 0.2) (layer "F.Cu") (net 6))
+  (segment (start 109.147601 57.099599) (end 108.241702 57.099599) (width 0.2) (layer "F.Cu") (net 6))
   (segment (start 119.65819 56.857389) (end 119.413801 56.613) (width 0.2) (layer "F.Cu") (net 6))
-  (segment (start 119.413801 56.613) (end 115.4092 56.613) (width 0.2) (layer "F.Cu") (net 6))
-  (segment (start 108.216701 57.1246) (end 107.6452 57.1246) (width 0.2) (layer "F.Cu") (net 6))
-  (segment (start 112.8692 59.153) (end 111.201002 59.153) (width 0.2) (layer "F.Cu") (net 6))
+  (segment (start 114.7282 58.6656) (end 114.2408 59.153) (width 0.2) (layer "F.Cu") (net 6))
+  (segment (start 114.2408 59.153) (end 111.201002 59.153) (width 0.2) (layer "F.Cu") (net 6))
+  (segment (start 115.4092 56.613) (end 114.7282 57.294) (width 0.2) (layer "F.Cu") (net 6))
+  (segment (start 114.7282 57.294) (end 114.7282 58.6656) (width 0.2) (layer "F.Cu") (net 6))
   (segment (start 108.241702 57.099599) (end 108.216701 57.1246) (width 0.2) (layer "F.Cu") (net 6))
-  (segment (start 109.147601 57.099599) (end 108.241702 57.099599) (width 0.2) (layer "F.Cu") (net 6))
   (via (at 119.65819 56.99881) (size 0.4) (drill 0.3) (layers "F.Cu" "B.Cu") (net 6))
   (segment (start 119.1549 58.5909) (end 119.254901 58.490899) (width 0.2) (layer "B.Cu") (net 6))
@@
   (segment (start 120.1549 57.3541) (end 120.0464 57.2456) (width 0.2) (layer "B.Cu") (net 6))
   (segment (start 119.1549 59.5159) (end 119.1549 58.5909) (width 0.2) (layer "B.Cu") (net 6))
+  (segment (start 108.241702 56.649599) (end 108.216701 56.624598) (width 0.2) (layer "F.Cu") (net 7))
   (segment (start 109.481599 56.649599) (end 108.241702 56.649599) (width 0.2) (layer "F.Cu") (net 7))
+  (segment (start 108.216701 56.624598) (end 107.6452 56.624598) (width 0.2) (layer "F.Cu") (net 7))
   (segment (start 111.535 58.703) (end 109.481599 56.649599) (width 0.2) (layer "F.Cu") (net 7))
-  (segment (start 112.6828 58.703) (end 111.535 58.703) (width 0.2) (layer "F.Cu") (net 7))
+  (segment (start 119.600199 56.163) (end 115.2228 56.163) (width 0.2) (layer "F.Cu") (net 7))
+  (segment (start 114.0544 58.703) (end 111.535 58.703) (width 0.2) (layer "F.Cu") (net 7))
+  (segment (start 114.2782 57.1076) (end 114.2782 58.4792) (width 0.2) (layer "F.Cu") (net 7))
+  (segment (start 115.2228 56.163) (end 114.2782 57.1076) (width 0.2) (layer "F.Cu") (net 7))
+  (segment (start 120.11781 56.53919) (end 119.976389 56.53919) (width 0.2) (layer "F.Cu") (net 7))
   (segment (start 119.976389 56.53919) (end 119.600199 56.163) (width 0.2) (layer "F.Cu") (net 7))
-  (segment (start 108.216701 56.624598) (end 107.6452 56.624598) (width 0.2) (layer "F.Cu") (net 7))
-  (segment (start 120.11781 56.53919) (end 119.976389 56.53919) (width 0.2) (layer "F.Cu") (net 7))
-  (segment (start 108.241702 56.649599) (end 108.216701 56.624598) (width 0.2) (layer "F.Cu") (net 7))
-  (segment (start 119.600199 56.163) (end 115.2228 56.163) (width 0.2) (layer "F.Cu") (net 7))
-  (segment (start 115.2228 56.163) (end 112.6828 58.703) (width 0.2) (layer "F.Cu") (net 7))
+  (segment (start 114.2782 58.4792) (end 114.0544 58.703) (width 0.2) (layer "F.Cu") (net 7))
   (via (at 120.11781 56.53919) (size 0.4) (drill 0.3) (layers "F.Cu" "B.Cu") (net 7))
   (segment (start 120.6299 59.4909) (end 120.6549 59.5159) (width 0.2) (layer "B.Cu") (net 7))
